Commit message: Lab 2 - gazebo working

File: turtle_bot/control/gazebo_control.xacro (robot description, xacro)
@@ -11,4 +11,6 @@
             <max_wheel_torque>200</max_wheel_torque>
             <max_wheel_acceleration>10.0</max_wheel_acceleration>
+            <!--Input-->
+            <topic>cmd_vel</topic>
             <!--outputs-->
             <frame_id>odom</frame_id>

File: turtle_bot/macros/wheels.xacro (robot description, xacro)
@@ -1,10 +1,10 @@
 <?xml version="1.0"?>
 <robot xmlns:xacro="http://www.ros.org/wiki/xacro">
-        <xacro:macro name="wheel" params="wheel_number wheel_mass *origin *parent">
+        <xacro:macro name="wheel" params="wheel_number wheel_mass reflect *origin *parent">
             <joint name = "wheel_joint_${wheel_number}" type="continuous">
                     <xacro:insert_block name="origin"/>
                     <xacro:insert_block name="parent"/>
                     <child link="wheel_${wheel_number}"/>
-                    <axis xyz="0 0 1">
+                    <axis xyz="0 0 ${reflect * 1}">
                             <limit>
                                     <effort>20</effort>
@@ -43,3 +43,37 @@
             </gazebo>
         </xacro:macro>
+        <xacro:macro name="caster_wheel" params="wheel_mass *origin *parent">
+                <joint name = "caster_wheel_joint" type="fixed">
+                    <xacro:insert_block name="origin"/>
+                    <xacro:insert_block name="parent"/>
+                    <child link="caster_wheel"/>
+                </joint>
+                <link name="caster_wheel">
+                    <visual name="caster_wheel_visual">
+                        <origin xyz="0 0 -0.0097931037703787721105" rpy="0 -0 0" />
+                        <geometry>
+                               <sphere radius="${caster_wheel_radius}"/>
+                        </geometry>
+                        <material name="grey_wheel"/>
+                    </visual>
+                    <collision name="caster_wheel_collision">
+                        <origin xyz="0 0 -0.0097931037703787721105" rpy="0 -0 0" />
+                        <geometry>
+                               <sphere radius="${caster_wheel_radius}"/>
+                        </geometry>
+                    </collision>
+                    <xacro:wheel_inertial  mass="${wheel_mass}">
+                        <origin xyz="-9.1775008443145391876e-19 -6.7665573084812139498e-22 -0.0099999999999999932693" rpy="0 0 0"/>
+                        <inertia ixx="1.3557884731460580961e-05" ixy="0"  ixz="0" iyy="1.3557884731460580961e-05" iyz="0" izz="2.3145947892207558913e-05" />
+                    </xacro:wheel_inertial>
+                </link>
+                <!--Gazebo Material-->
+                <gazebo reference="caster_wheel">
+                    <material>Gazebo/Gray</material>
+                    <!--Friction Coefficients-->
+                    <!--Making it frictionless-->
+                    <mu1>0.001</mu1>
+                    <mu2>0.001</mu2>
+                </gazebo>
+        </xacro:macro>
 </robot>

File: turtle_bot/turtle_bot_core.xacro (robot description, xacro)
@@ -13,4 +13,5 @@
     <xacro:property name="lidar_mass" value="0.19842109046142830664"/>
     <xacro:property name="wheel_torque" value="20"/>
+    <xacro:property name="caster_wheel_radius" value="0.017"/>
     <!--BASE LAYER-->
     <link name="base_layer">
@@ -127,12 +128,17 @@
     <!--WHEELS-->
     <!--LEFT_WHEELS-->
-    <xacro:wheel wheel_number="1" wheel_mass="${wheel_mass}">
+    <xacro:wheel wheel_number="1" wheel_mass="${wheel_mass}" reflect="1">
         <origin xyz="0.080330040283809592272 0.0063858766431100638661 -0.01323314544227911782" rpy="-0 1.570796326794896558 0"/>
         <parent link="base_layer"/>
     </xacro:wheel>
     <!--RIGHT_WHEEL-->
-    <xacro:wheel wheel_number="2" wheel_mass="${wheel_mass}">
+    <xacro:wheel wheel_number="2" wheel_mass="${wheel_mass}" reflect="-1">
         <origin xyz="-0.091147230564865622249 0.0063858766431100638661 -0.01323314544227911782" rpy="-0 -1.570796326794896558 0"/>
         <parent link="base_layer"/>
     </xacro:wheel>
+    <!--CASTER WHEEL-->
+    <xacro:caster_wheel wheel_mass="${wheel_mass}">
+        <origin xyz="0.005405 0.03 -0.01323" rpy="0 0 0"/>
+        <parent link="base_layer"/>
+    </xacro:caster_wheel>
 </robot>
